File: kicad-project/test/test.kicad_pcb (KiCad board)
At the start: 2 copper layers, 20 parts

Commit message: kicad 2 лаба
Parts:
- removed BF1: ЗП-25, Battery_Holders:Keystone_1042_1x18650
- added LS1: Speaker, Battery_Holders:Seiko_MS621F, F.Cu at (158.3, 110.8)
- moved C1 71.2 mm to (185.2, 113.3)
- moved R9 39.2 mm to (187.5, 108.0)
- moved C4 35.9 mm to (181.6, 118.8)
- moved R4 35.3 mm to (183.6, 108.0)
- moved VD2 35.1 mm to (177.9, 124.2)
- moved R6 33.8 mm to (181.3, 113.5)
- moved R1 32.0 mm to (177.4, 118.8)
- moved R7 31.7 mm to (180.1, 108.0)
- moved VD1 31.1 mm to (172.5, 124.8)
- moved R2 28.5 mm to (173.5, 118.8)
- moved R8 27.6 mm to (167.7, 124.8)
- moved C2 26.7 mm to (175.0, 107.9)
- moved R3 26.7 mm to (173.8, 113.3)
- moved C3 24.0 mm to (162.2, 124.7)
- moved VT1 23.2 mm to (167.4, 118.3)
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Connections:
- C3 pad 2: (no net) -> Net-(C3-Pad2)
